File: ACIR_PCB.kicad_pcb (KiCad board)
At the start: 2 copper layers, 297 x 210 mm, 39 parts, among them J1 TestPoint, J10 TestPoint, J11 TestPoint, J12 TestPoint, J13 TestPoint, J14 TestPoint, J15 TestPoint, J16 TestPoint, J17 TestPoint, J18 TestPoint, J19 TestPoint, J2 TestPoint, J20 TestPoint, J3 TestPoint, J4 TestPoint, J5 TestPoint, J6 TestPoint, J7 TestPoint, J8 TestPoint, J9 TestPoint

Commit message: Production verification complete: restore 1S 4P and 4S 1P header titles, audit silkscreen clearances, and generate production Gerbers and drill package
Other:
- board text added: "1S 4P"
Changed lines of the file:
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@@
+		)
+	)
+	(gr_text "4S 1P"
+		(at 268 119.66 0)
+		(layer "F.SilkS" knockout)
+		(effects
+			(font
+				(face "PT Sans")
+				(size 6 6)
+				(thickness 1.5)
+				(bold yes)
+			)
+		)
+		(render_cache "4S 1P" 0
+			(polygon
+				(pts
+					(xy 261.272819 119.641137) (xy 262.196057 119.641137) (xy 262.196057 120.555582) (xy 261.272819 120.555582)
+					(xy 261.272819 122.15) (xy 260.257257 122.15) (xy 260.257257 120.555582) (xy 257.71359 120.555582)
+					(xy 257.71359 119.892829) (xy 257.847876 119.708548) (xy 258.721092 119.708548) (xy 259.258182 119.641137)
+					(xy 260.257257 119.641137) (xy 260.257257 118.362159) (xy 260.332728 117.659839) (xy 260.299023 117.659839)
+					(xy 260.013991 118.261775) (xy 259.140945 119.390177) (xy 258.721092 119.708548) (xy 257.847876 119.708548)
+					(xy 260.374494 116.241277) (xy 261.272819 116.241277)
+				)
+			)
+			(polygon
+				(pts
+					(xy 265.352651 120.551552) (xy 265.330208 120.385144) (xy 265.265158 120.244539) (xy 265.155181 120.123272)
+					(xy 264.940632 119.970424) (xy 264.659857 119.822487) (xy 264.01359 119.539654) (xy 263.676891 119.374993)
+					(xy 263.367323 119.178053) (xy 263.095263 118.938194) (xy 262.871999 118.64426) (xy 262.766458 118.422899)
+					(xy 262.69907 118.154526) (xy 262.674895 117.828733) (xy 262.712488 117.418388) (xy 262.817411 117.085013)
+					(xy 262.991257 116.795117) (xy 263.224441 116.559647) (xy 263.509085 116.378716) (xy 263.849825 116.248604)
+					(xy 264.223242 116.173871) (xy 264.655827 116.147487) (xy 265.159424 116.17088) (xy 265.621196 116.238712)
+					(xy 266.049336 116.355463) (xy 266.368213 116.502861) (xy 266.007344 117.489846) (xy 265.796549 117.38541)
+					(xy 265.453402 117.275889) (xy 265.075045 117.204044) (xy 264.655827 117.179169) (xy 264.390731 117.199349)
+					(xy 264.189769 117.253617) (xy 264.038869 117.335607) (xy 263.919112 117.452785) (xy 263.849043 117.590273)
+					(xy 263.824912 117.755094) (xy 263.846813 117.910391) (xy 263.911254 118.045682) (xy 264.022016 118.166521)
+					(xy 264.236591 118.319947) (xy 264.517341 118.470969) (xy 265.163607 118.761863) (xy 265.50072 118.929683)
+					(xy 265.809874 119.127494) (xy 266.082433 119.366688) (xy 266.305198 119.657257) (xy 266.411624 119.87557)
+					(xy 266.4788 120.134578) (xy 266.502669 120.443108) (xy 266.461532 120.893103) (xy 266.34733 121.254239)
+					(xy 266.159576 121.567469) (xy 265.910624 121.821737) (xy 265.605895 122.016299) (xy 265.231018 122.157693)
+					(xy 264.820498 122.238835) (xy 264.353942 122.267236) (xy 263.744339 122.234953) (xy 263.24569 122.145969)
+					(xy 262.801522 122.014322) (xy 262.540806 121.90307) (xy 262.910101 120.899965) (xy 263.149337 121.009141)
+					(xy 263.480896 121.118318) (xy 263.871074 121.202215) (xy 264.294958 121.235554) (xy 264.634283 121.213435)
+					(xy 264.889874 121.154407) (xy 265.07971 121.06666) (xy 265.230897 120.934921) (xy 265.320868 120.76719)
+				)
+			)
+			(polygon
+				(pts
+					(xy 269.732903 121.235554) (xy 270.899773 121.235554) (xy 270.899773 117.912997) (xy 271.025802 117.341102)
+					(xy 270.622801 117.837892) (xy 269.875418 118.351535) (xy 269.413799 117.719923) (xy 271.327686 116.170935)
+					(xy 271.940614 116.170935) (xy 271.940614 121.235554) (xy 273.082205 121.235554) (xy 273.082205 122.15)
+					(xy 269.732903 122.15)
+				)
+			)
+			(polygon
+				(pts
+					(xy 276.204988 116.212144) (xy 276.64583 116.265823) (xy 277.068363 116.37392) (xy 277.439009 116.550488)
+					(xy 277.657883 116.709925) (xy 277.849073 116.906943) (xy 278.014201 117.145464) (xy 278.132378 117.408794)
+					(xy 278.208867 117.734928) (xy 278.236584 118.137944) (xy 278.213115 118.502596) (xy 278.147161 118.811011)
+					(xy 278.04351 119.072173) (xy 277.816949 119.421069) (xy 277.531332 119.696092) (xy 277.192686 119.904465)
+					(xy 276.805198 120.048168) (xy 276.392615 120.129546) (xy 275.961828 120.156978) (xy 275.827372 120.156978)
+					(xy 275.634298 120.152948) (xy 275.437194 120.140125) (xy 275.298709 120.123272) (xy 275.298709 122.15)
+					(xy 274.148691 122.15) (xy 274.148691 117.198953) (xy 275.298709 117.198953) (xy 275.298709 119.1612)
+					(xy 275.399459 119.178419) (xy 275.541974 119.191242) (xy 275.688887 119.195638) (xy 275.794033 119.195638)
+					(xy 276.242829 119.152407) (xy 276.455685 119.09016) (xy 276.6418 118.992672) (xy 276.798521 118.855066)
+					(xy 276.922801 118.66844) (xy 276.999033 118.441777) (xy 277.027948 118.123656) (xy 277.000778 117.854394)
+					(xy 276.927198 117.652878) (xy 276.80965 117.484092) (xy 276.662683 117.354658) (xy 276.489416 117.260232)
+					(xy 276.289358 117.198953) (xy 275.861078 117.155722) (xy 275.541974 117.168911) (xy 275.298709 117.198953)
+					(xy 274.148691 117.198953) (xy 274.148691 116.336898) (xy 274.925017 116.232117) (xy 275.768754 116.194382)
+				)
+			)
+		)
+	)
+	(gr_text "1S 4P"
+		(at 125.18 119.66 0)
+		(layer "F.SilkS" knockout)
+		(effects
+			(font
+				(face "PT Sans")
+				(size 6 6)
+				(thickness 1.5)
+				(bold yes)
+			)
+		)
+		(render_cache "1S 4P" 0
+			(polygon
+				(pts
+					(xy 115.581988 121.235554) (xy 116.748859 121.235554) (xy 116.748859 117.912997) (xy 116.874888 117.341102)
+					(xy 116.471887 117.837892) (xy 115.724504 118.351535) (xy 115.262885 117.719923) (xy 117.176772 116.170935)
+					(xy 117.7897 116.170935) (xy 117.7897 121.235554) (xy 118.931291 121.235554) (xy 118.931291 122.15)
+					(xy 115.581988 122.15)
+				)
+			)
+			(polygon
+				(pts
+					(xy 122.532651 120.551552) (xy 122.510208 120.385144) (xy 122.445158 120.244539) (xy 122.335181 120.123272)
+					(xy 122.120632 119.970424) (xy 121.839857 119.822487) (xy 121.19359 119.539654) (xy 120.856891 119.374993)
+					(xy 120.547323 119.178053) (xy 120.275263 118.938194) (xy 120.051999 118.64426) (xy 119.946458 118.422899)
+					(xy 119.87907 118.154526) (xy 119.854895 117.828733) (xy 119.892488 117.418388) (xy 119.997411 117.085013)
+					(xy 120.171257 116.795117) (xy 120.404441 116.559647) (xy 120.689085 116.378716) (xy 121.029825 116.248604)
+					(xy 121.403242 116.173871) (xy 121.835827 116.147487) (xy 122.339424 116.17088) (xy 122.801196 116.238712)
+					(xy 123.229336 116.355463) (xy 123.548213 116.502861) (xy 123.187344 117.489846) (xy 122.976549 117.38541)
+					(xy 122.633402 117.275889) (xy 122.255045 117.204044) (xy 121.835827 117.179169) (xy 121.570731 117.199349)
+					(xy 121.369769 117.253617) (xy 121.218869 117.335607) (xy 121.099112 117.452785) (xy 121.029043 117.590273)
+					(xy 121.004912 117.755094) (xy 121.026813 117.910391) (xy 121.091254 118.045682) (xy 121.202016 118.166521)
+					(xy 121.416591 118.319947) (xy 121.697341 118.470969) (xy 122.343607 118.761863) (xy 122.68072 118.929683)
+					(xy 122.989874 119.127494) (xy 123.262433 119.366688) (xy 123.485198 119.657257) (xy 123.591624 119.87557)
+					(xy 123.6588 120.134578) (xy 123.682669 120.443108) (xy 123.641532 120.893103) (xy 123.52733 121.254239)
+					(xy 123.339576 121.567469) (xy 123.090624 121.821737) (xy 122.785895 122.016299) (xy 122.411018 122.157693)
+					(xy 122.000498 122.238835) (xy 121.533942 122.267236) (xy 120.924339 122.234953) (xy 120.42569 122.145969)
+					(xy 119.981522 122.014322) (xy 119.720806 121.90307) (xy 120.090101 120.899965) (xy 120.329337 121.009141)
+					(xy 120.660896 121.118318) (xy 121.051074 121.202215) (xy 121.474958 121.235554) (xy 121.814283 121.213435)
+					(xy 122.069874 121.154407) (xy 122.25971 121.06666) (xy 122.410897 120.934921) (xy 122.500868 120.76719)
+				)
+			)
+			(polygon
+				(pts
+					(xy 129.783733 119.641137) (xy 130.706971 119.641137) (xy 130.706971 120.555582) (xy 129.783733 120.555582)
+					(xy 129.783733 122.15) (xy 128.768171 122.15) (xy 128.768171 120.555582) (xy 126.224504 120.555582)
+					(xy 126.224504 119.892829) (xy 126.35879 119.708548) (xy 127.232006 119.708548) (xy 127.769096 119.641137)
+					(xy 128.768171 119.641137) (xy 128.768171 118.362159) (xy 128.843642 117.659839) (xy 128.809937 117.659839)
+					(xy 128.524905 118.261775) (xy 127.651859 119.390177) (xy 127.232006 119.708548) (xy 126.35879 119.708548)
+					(xy 128.885408 116.241277) (xy 129.783733 116.241277)
+				)
+			)
+			(polygon
+				(pts
+					(xy 133.384988 116.212144) (xy 133.82583 116.265823) (xy 134.248363 116.37392) (xy 134.619009 116.550488)
+					(xy 134.837883 116.709925) (xy 135.029073 116.906943) (xy 135.194201 117.145464) (xy 135.312378 117.408794)
+					(xy 135.388867 117.734928) (xy 135.416584 118.137944) (xy 135.393115 118.502596) (xy 135.327161 118.811011)
+					(xy 135.22351 119.072173) (xy 134.996949 119.421069) (xy 134.711332 119.696092) (xy 134.372686 119.904465)
+					(xy 133.985198 120.048168) (xy 133.572615 120.129546) (xy 133.141828 120.156978) (xy 133.007372 120.156978)
+					(xy 132.814298 120.152948) (xy 132.617194 120.140125) (xy 132.478709 120.123272) (xy 132.478709 122.15)
+					(xy 131.328691 122.15) (xy 131.328691 117.198953) (xy 132.478709 117.198953) (xy 132.478709 119.1612)
+					(xy 132.579459 119.178419) (xy 132.721974 119.191242) (xy 132.868887 119.195638) (xy 132.974033 119.195638)
+					(xy 133.422829 119.152407) (xy 133.635685 119.09016) (xy 133.8218 118.992672) (xy 133.978521 118.855066)
+					(xy 134.102801 118.66844) (xy 134.179033 118.441777) (xy 134.207948 118.123656) (xy 134.180778 117.854394)
+					(xy 134.107198 117.652878) (xy 133.98965 117.484092) (xy 133.842683 117.354658) (xy 133.669416 117.260232)
+					(xy 133.469358 117.198953) (xy 133.041078 117.155722) (xy 132.721974 117.168911) (xy 132.478709 117.198953)
+					(xy 131.328691 117.198953) (xy 131.328691 116.336898) (xy 132.105017 116.232117) (xy 132.948754 116.194382)
+				)
+			)
 		)
 	)
