File: ACIR_PCB.kicad_pcb (KiCad board)
At the start: 2 copper layers, 297 x 210 mm, 39 parts, among them J1 TestPoint, J10 TestPoint, J11 TestPoint, J12 TestPoint, J13 TestPoint, J14 TestPoint, J15 TestPoint, J16 TestPoint, J17 TestPoint, J18 TestPoint, J19 TestPoint, J2 TestPoint, J20 TestPoint, J3 TestPoint, J4 TestPoint, J5 TestPoint, J6 TestPoint, J7 TestPoint, J8 TestPoint, J9 TestPoint

Commit message: feat: add test points to PCB layout and generate production and Gerber files
Routing:
- net Net-(BT2--): vias 196 -> 198
- net (no net): vias 0 -> 186

Commit message: refactor: replace through-hole test points with SMD pads in PCB layout
Parts:
- J1, J10, J11, J12, J13, J14, J15, J16, J17, J18, J19, J2, J20, J3, J4, J5, J6, J7, J8, J9: footprint TestPoint:TestPoint_Bridge_Pitch2.54mm_Drill1.3mm -> TestPoint:TestPoint_Pad_D2.0mm
- moved J10 3.89 mm to (178.7, 139.3), turned to 0 degrees
- moved J11 3.89 mm to (74.4, 139.3), turned to 0 degrees
- moved J12 3.89 mm to (178.7, 163.0), turned to 0 degrees
- moved J13 3.89 mm to (74.4, 163.0), turned to 0 degrees
- moved J14 3.89 mm to (178.7, 186.8), turned to 0 degrees
- moved J15 3.89 mm to (74.4, 186.8), turned to 0 degrees
- moved J16 3.89 mm to (178.7, 210.5), turned to 0 degrees
- moved J17 3.89 mm to (74.4, 210.5), turned to 0 degrees
- moved J1 2.00 mm to (249.6, 87.2), turned to 0 degrees
- moved J2 2.00 mm to (145.2, 87.2), turned to 0 degrees
- moved J18 1.27 mm to (216.0, 163.0), turned to 0 degrees
- moved J19 1.27 mm to (320.4, 186.8), turned to 0 degrees
- moved J20 1.27 mm to (216.0, 210.5), turned to 0 degrees
- moved J3 1.27 mm to (320.4, 139.3), turned to 0 degrees
- moved J4 1.27 mm to (320.4, 210.5), turned to 0 degrees
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Routing:
- net /4P_B-: track 456.5 -> 478.6 mm, vias 462 -> 797
- net /4P_B+: track 460.3 -> 482.4 mm, vias 470 -> 797
- net /1S_B-: track 68.9 -> 72.0 mm, vias 62 -> 121
- net /1S_B+: track 68.9 -> 72.0 mm, vias 60 -> 121
- net Net-(BT4--): vias 196 -> 341
- net Net-(BT3--): vias 202 -> 336
- net Net-(BT2--): vias 198 -> 341
- net /4S_B-: vias 72 -> 121
- net /4S_B+: vias 72 -> 121

Commit message: chore: clean up test artifacts and generate production gerbers and manufacturing files
Parts:
- BT1, BT2, BT3, BT4, BT5, BT6, BT7, BT8, BT9: value BH18650B1BA002 -> BH-18650-B5BA008
- H1, H2, H3, H4, H5, H6, H7, H8: value MountingHole_Pad -> MountingHole_M3_Pad
- J1, J10: value TestPoint -> 1S 1P +ve
- J11, J18, J2: value TestPoint -> 1S 1P -ve
- J12: value TestPoint -> 1S 3P +ve
- J13: value TestPoint -> 1S 3P -ve
- J14: value TestPoint -> 1S 4P +ve
- J15: value TestPoint -> 1S 4P -ve
- J16: value TestPoint -> 1S 2P +ve
- J17: value TestPoint -> 1S 2P -ve
- J19: value TestPoint -> 2S 1P -ve
- J20: value TestPoint -> 3S 1P -ve
- J3: value TestPoint -> 4S B +ve
- J4: value TestPoint -> 4S B -ve
- J5: value TestPoint -> 4P B +ve
- J6: value TestPoint -> 4P B -ve
- J7: value TestPoint -> 2S 1P +ve
- J8: value TestPoint -> 3S 1P +ve
- J9: value TestPoint -> 4S 1P +ve
Routing:
- net /4P_B+: track 482.4 -> 478.6 mm
- net (no net): vias 186 -> 0
Other:
- board text added: "BT1 +ve"
- board text added: "BT1 -ve"
- board text added: "BT2"
- board text added: "BT2 +ve"
- board text added: "BT3"
- board text added: "BT4"
- board text added: "BT5"
- board text added: "BT5 -ve"
- board text added: "BT6 +ve"
- board text added: "BT6 -ve"
- board text added: "BT7 +ve"
- board text added: "BT7 -ve"
- board text added: "BT8 +ve"
- board text added: "BT8 -ve"
- board text added: "BT9 +ve"
- board text added: "BT9 -ve"
- board text removed: "1S 1P +ve"
- board text removed: "1S 1P -ve"
- board text removed: "1S 2P +ve"
- board text removed: "1S 2P -ve"
- board text removed: "1S 3P +ve"
- board text removed: "1S 3P -ve"
- board text removed: "1S 4P +ve"
- board text removed: "1S 4P -ve"
- board text removed: "2S 1P"
- board text removed: "3S 1P"
- board text removed: "4S 1P -ve"

Commit message: chore: generate gerbers and production manufacturing files for PCB layout
Other:
- board text added: "BT1"
- board text added: "BT6"
- board text added: "BT7"
- board text added: "BT8"
- board text added: "BT9"
- board text added: "Designed by Ashutosh Raj, Shreyas P & Suraj S D"
- board text added: "Product ID: TST-ACR-V1.1-2607 Sub product ID: TST-ACR-V1.1-L1-2607 Version: V1.1"
- board text added: "TST-ACIR-V1.1-2608-0"
- board text removed: "BT1 +ve"
- board text removed: "BT1 -ve"
- board text removed: "BT2 +ve"
- board text removed: "BT5 -ve"
- board text removed: "BT6 +ve"
- board text removed: "BT6 -ve"
- board text removed: "BT7 +ve"
- board text removed: "BT7 -ve"
- board text removed: "BT8 +ve"
- board text removed: "BT8 -ve"
- board text removed: "BT9 +ve"
- board text removed: "BT9 -ve"
- board text removed: "Product ID: TST-ACR-V1-2607 Sub product ID: TST-ACR-V1-L1-2607 Version: V1"
