File: test_diag.kicad_sch (KiCad schematic)
At the start: 37 parts, among them J1 1S 1P +ve, J10 1S 1P +ve, J11 1S 1P -ve, J12 1S 3P +ve, J13 1S 3P -ve, J14 1S 4P +ve, J15 1S 4P -ve, J16 1S 2P +ve, J17 1S 2P -ve, J18 1S 1P -ve, J19 2S 1P -ve, J2 1S 1P -ve, J20 3S 1P -ve, J3 4S B +ve, J4 4S B -ve, J5 4P B +ve, J6 4P B -ve, J7 2S 1P +ve, J8 3S 1P +ve, J9 4S 1P +ve

Commit message: test: add test schematics, ERC reports, and verification artifacts for ACIR PCB
Parts:
- removed H2, H3, H4, H5, H6, H7, H8: MountingHole_M3_Pad, footprints:MountingHole_3.2mm_M3, symbol Mechanical:MountingHole
