File: test_fix_all.kicad_sch (KiCad schematic)
At the start: 37 parts, among them J1 1S 1P +ve, J10 1S 1P +ve, J11 1S 1P -ve, J12 1S 3P +ve, J13 1S 3P -ve, J14 1S 4P +ve, J15 1S 4P -ve, J16 1S 2P +ve, J17 1S 2P -ve, J18 1S 1P -ve, J19 2S 1P -ve, J2 1S 1P -ve, J20 3S 1P -ve, J3 4S B +ve, J4 4S B -ve, J5 4P B +ve, J6 4P B -ve, J7 2S 1P +ve, J8 3S 1P +ve, J9 4S 1P +ve

Commit message: test: add test schematics, ERC reports, and verification artifacts for ACIR PCB
Changed lines of the file:
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@@
 		(fields_autoplaced yes)
 		(property "Reference" "H1"
-			(at 223.81 151.13 0)
+			(at 220.00 149.86 0)
 			(show_name no)
 			(do_not_autoplace no)
@@
 		)
 		(property "Value" "MountingHole_M3_Pad"
-			(at 223.81 153.67 0)
+			(at 220.00 154.94 0)
 			(show_name no)
 			(do_not_autoplace no)
@@
 		(fields_autoplaced yes)
 		(property "Reference" "H2"
-			(at 223.81 163.83 0)
+			(at 220.00 162.56 0)
 			(show_name no)
 			(do_not_autoplace no)
@@
 		)
 		(property "Value" "MountingHole_M3_Pad"
-			(at 223.81 166.37 0)
+			(at 220.00 167.64 0)
 			(show_name no)
 			(do_not_autoplace no)
@@
 		(fields_autoplaced yes)
 		(property "Reference" "H3"
-			(at 223.81 176.53 0)
+			(at 220.00 175.26 0)
 			(show_name no)
 			(do_not_autoplace no)
@@
 		)
 		(property "Value" "MountingHole_M3_Pad"
-			(at 223.81 179.07 0)
+			(at 220.00 180.34 0)
 			(show_name no)
 			(do_not_autoplace no)
@@
 		(fields_autoplaced yes)
 		(property "Reference" "H4"
-			(at 223.81 189.23 0)
+			(at 220.00 187.96 0)
 			(show_name no)
 			(do_not_autoplace no)
@@
 		)
 		(property "Value" "MountingHole_M3_Pad"
-			(at 223.81 191.77 0)
+			(at 220.00 193.04 0)
 			(show_name no)
 			(do_not_autoplace no)
@@
 		(fields_autoplaced yes)
 		(property "Reference" "H5"
-			(at 273.81 151.13 0)
+			(at 270.00 149.86 0)
 			(show_name no)
 			(do_not_autoplace no)
@@
 		)
 		(property "Value" "MountingHole_M3_Pad"
-			(at 273.81 153.67 0)
+			(at 270.00 154.94 0)
 			(show_name no)
 			(do_not_autoplace no)
@@
 		(fields_autoplaced yes)
 		(property "Reference" "H6"
-			(at 273.81 163.83 0)
+			(at 270.00 162.56 0)
 			(show_name no)
 			(do_not_autoplace no)
@@
 		)
 		(property "Value" "MountingHole_M3_Pad"
-			(at 273.81 166.37 0)
+			(at 270.00 167.64 0)
 			(show_name no)
 			(do_not_autoplace no)
@@
 		(fields_autoplaced yes)
 		(property "Reference" "H7"
-			(at 273.81 176.53 0)
+			(at 270.00 175.26 0)
 			(show_name no)
 			(do_not_autoplace no)
@@
 		)
 		(property "Value" "MountingHole_M3_Pad"
-			(at 273.81 179.07 0)
+			(at 270.00 180.34 0)
 			(show_name no)
 			(do_not_autoplace no)
@@
 		(fields_autoplaced yes)
 		(property "Reference" "H8"
-			(at 273.81 189.23 0)
+			(at 270.00 187.96 0)
 			(show_name no)
 			(do_not_autoplace no)
@@
 		)
 		(property "Value" "MountingHole_M3_Pad"
-			(at 273.81 191.77 0)
-			(show_name no)
-			(do_not_autoplace no)
+			(at 270.00 193.04 0)
+			(show_name no)
+			(do_not_autoplace no)
