File: ACIR-Learning-Kit-1-PCB/ACIR-Learning-Kit-1-PCB.kicad_sch (KiCad schematic)
At the start: 37 parts, among them J1 1S 1P +ve, J10 1S 1P +ve, J11 1S 1P -ve, J12 1S 3P +ve, J13 1S 3P -ve, J14 1S 4P +ve, J15 1S 4P -ve, J16 1S 2P +ve, J17 1S 2P -ve, J18 1S 1P -ve, J19 2S 1P -ve, J2 1S 1P -ve, J20 3S 1P -ve, J3 4S B +ve, J4 4S B -ve, J5 4P B +ve, J6 4P B -ve, J7 2S 1P +ve, J8 3S 1P +ve, J9 4S 1P +ve

Commit message: feat: DFM optimization - clean circular probing pads, uniform 2.0mm via pitch, and zero warnings
Parts:
- J1, J10, J11, J12, J13, J14, J15, J16, J17, J18, J19, J2, J20, J3, J4, J5, J6, J7, J8, J9: footprint TestPoint:TestPoint_Pad_D2.0mm -> footprints:TestPoint_Pad_D6.0mm
Changed lines of the file:
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@@
 			)
 		)
-		(property "Footprint" "TestPoint:TestPoint_Pad_D2.0mm"
+		(property "Footprint" "footprints:TestPoint_Pad_D6.0mm"
 			(at 137.16 207.01 0)
 			(hide yes)
@@
 			)
 		)
-		(property "Footprint" "TestPoint:TestPoint_Pad_D2.0mm"
+		(property "Footprint" "footprints:TestPoint_Pad_D6.0mm"
 			(at 154.94 53.34 0)
 			(hide yes)
@@
 			)
 		)
-		(property "Footprint" "TestPoint:TestPoint_Pad_D2.0mm"
+		(property "Footprint" "footprints:TestPoint_Pad_D6.0mm"
 			(at 261.62 99.06 0)
 			(hide yes)
@@
 			)
 		)
-		(property "Footprint" "TestPoint:TestPoint_Pad_D2.0mm"
+		(property "Footprint" "footprints:TestPoint_Pad_D6.0mm"
 			(at 101.6 142.24 0)
 			(hide yes)
@@
 			)
 		)
-		(property "Footprint" "TestPoint:TestPoint_Pad_D2.0mm"
+		(property "Footprint" "footprints:TestPoint_Pad_D6.0mm"
 			(at 66.04 186.69 0)
 			(hide yes)
@@
 			)
 		)
-		(property "Footprint" "TestPoint:TestPoint_Pad_D2.0mm"
+		(property "Footprint" "footprints:TestPoint_Pad_D6.0mm"
 			(at 101.6 233.68 0)
 			(hide yes)
@@
 			)
 		)
-		(property "Footprint" "TestPoint:TestPoint_Pad_D2.0mm"
+		(property "Footprint" "footprints:TestPoint_Pad_D6.0mm"
 			(at 66.04 207.01 0)
 			(hide yes)
@@
 			)
 		)
-		(property "Footprint" "TestPoint:TestPoint_Pad_D2.0mm"
+		(property "Footprint" "footprints:TestPoint_Pad_D6.0mm"
 			(at 312.42 99.06 0)
 			(hide yes)
@@
 			)
 		)
-		(property "Footprint" "TestPoint:TestPoint_Pad_D2.0mm"
+		(property "Footprint" "footprints:TestPoint_Pad_D6.0mm"
 			(at 137.16 166.37 0)
 			(hide yes)
@@
 			)
 		)
-		(property "Footprint" "TestPoint:TestPoint_Pad_D2.0mm"
+		(property "Footprint" "footprints:TestPoint_Pad_D6.0mm"
 			(at 73.66 83.82 0)
 			(hide yes)
@@
 			)
 		)
-		(property "Footprint" "TestPoint:TestPoint_Pad_D2.0mm"
+		(property "Footprint" "footprints:TestPoint_Pad_D6.0mm"
 			(at 312.42 43.18 0)
 			(hide yes)
@@
 			)
 		)
-		(property "Footprint" "TestPoint:TestPoint_Pad_D2.0mm"
+		(property "Footprint" "footprints:TestPoint_Pad_D6.0mm"
 			(at 363.22 99.06 0)
 			(hide yes)
@@
 			)
 		)
-		(property "Footprint" "TestPoint:TestPoint_Pad_D2.0mm"
+		(property "Footprint" "footprints:TestPoint_Pad_D6.0mm"
 			(at 261.62 43.18 0)
 			(hide yes)
@@
 			)
 		)
-		(property "Footprint" "TestPoint:TestPoint_Pad_D2.0mm"
+		(property "Footprint" "footprints:TestPoint_Pad_D6.0mm"
 			(at 210.82 43.18 0)
 			(hide yes)
@@
 			)
 		)
-		(property "Footprint" "TestPoint:TestPoint_Pad_D2.0mm"
+		(property "Footprint" "footprints:TestPoint_Pad_D6.0mm"
 			(at 137.16 186.69 0)
 			(hide yes)
@@
 			)
 		)
-		(property "Footprint" "TestPoint:TestPoint_Pad_D2.0mm"
+		(property "Footprint" "footprints:TestPoint_Pad_D6.0mm"
 			(at 363.22 43.18 0)
 			(hide yes)
@@
 			)
 		)
-		(property "Footprint" "TestPoint:TestPoint_Pad_D2.0mm"
+		(property "Footprint" "footprints:TestPoint_Pad_D6.0mm"
 			(at 154.94 88.9 0)
 			(hide yes)
@@
 			)
 		)
-		(property "Footprint" "TestPoint:TestPoint_Pad_D2.0mm"
+		(property "Footprint" "footprints:TestPoint_Pad_D6.0mm"
 			(at 210.82 99.06 0)
 			(hide yes)
@@
 			)
 		)
-		(property "Footprint" "TestPoint:TestPoint_Pad_D2.0mm"
+		(property "Footprint" "footprints:TestPoint_Pad_D6.0mm"
 			(at 66.04 166.37 0)
 			(hide yes)
@@
 			)
 		)
-		(property "Footprint" "TestPoint:TestPoint_Pad_D2.0mm"
+		(property "Footprint" "footprints:TestPoint_Pad_D6.0mm"
 			(at 73.66 45.72 0)
 			(hide yes)
