File: ACIR-Learning-Kit-1-PCB/ACIR-Learning-Kit-1-PCB.kicad_pcb (KiCad board)
At the start: 2 copper layers, 297 x 210 mm, 39 parts, among them J1 1S 1P +ve, J10 1S 1P +ve, J11 1S 1P -ve, J12 1S 3P +ve, J13 1S 3P -ve, J14 1S 4P +ve, J15 1S 4P -ve, J16 1S 2P +ve, J17 1S 2P -ve, J18 1S 1P -ve, J19 2S 1P -ve, J2 1S 1P -ve, J20 3S 1P -ve, J3 4S B +ve, J4 4S B -ve, J5 4P B +ve, J6 4P B -ve, J7 2S 1P +ve, J8 3S 1P +ve, J9 4S 1P +ve

Commit message: feat: add PCB design files for ACIR Learning Kits 1 and 2
Other:
- board text added: "P1"
- board text added: "P10"
- board text added: "P11"
- board text added: "P12"
- board text added: "P13"
- board text added: "P14"
- board text added: "P15"
- board text added: "P16"
- board text added: "P17"
- board text added: "P18"
- board text added: "P2"
- board text added: "P3"
- board text added: "P4"
- board text added: "P5"
- board text added: "P6"
- board text added: "P7"
- board text added: "P8"
- board text added: "P9"
- board text removed: "BT1"
- board text removed: "BT2"
- board text removed: "BT3"
- board text removed: "BT4"
- board text removed: "BT5"
- board text removed: "BT6"
- board text removed: "BT7"
- board text removed: "BT8"
- board text removed: "BT9"

Commit message: feat: add PCB design files, gerbers, and production outputs for ACIR Learning Kits 1 and 2
Parts:
- J1, J10, J11, J12, J13, J14, J15, J16, J17, J18, J19, J2, J20, J3, J4, J5, J6, J7, J8, J9: footprint TestPoint:TestPoint_Pad_D2.0mm -> footprints:TestPoint_Pad_D6.0mm
Routing:
- net /4P_B-: track 478.6 -> 470.2 mm, vias 797 -> 416
- net /4P_B+: track 478.6 -> 470.2 mm, vias 797 -> 416
- net Net-(BT4--): vias 341 -> 136
- net Net-(BT3--): vias 336 -> 136
- net Net-(BT2--): vias 341 -> 136
- net /4S_B-: vias 121 -> 26
- net /4S_B+: vias 121 -> 26
- net /1S_B-: vias 121 -> 26
- net /1S_B+: vias 121 -> 26
