File: ACIR-Learning-Kit-2-PCB/ACIR-Learning-Kit-2-PCB.kicad_sch (KiCad schematic)
At the start: 37 parts, among them J1 1S 1P +ve, J10 1S 1P +ve, J11 1S 1P -ve, J12 1S 3P +ve, J13 1S 3P -ve, J14 1S 4P +ve, J15 1S 4P -ve, J16 1S 2P +ve, J17 1S 2P -ve, J18 1S 1P -ve, J19 2S 1P -ve, J2 1S 1P -ve, J20 3S 1P -ve, J3 4S B +ve, J4 4S B -ve, J5 4P B +ve, J6 4P B -ve, J7 2S 1P +ve, J8 3S 1P +ve, J9 4S 1P +ve

Commit message: feat: add PCB design files for ACIR Learning Kits 1 and 2
Parts:
- removed BT1: BH-18650-B5BA008, footprints:BH18650B1BA002, symbol Device:Battery_Cell
- removed J5: 4P B +ve, TestPoint:TestPoint_Pad_D2.0mm, symbol Connector:Conn_01x01_Pin
- removed J6: 4P B -ve, TestPoint:TestPoint_Pad_D2.0mm, symbol Connector:Conn_01x01_Pin
- added J21, J23: 1S 1P +ve, TestPoint:TestPoint_Pad_D2.0mm, symbol Connector:Conn_01x01_Pin
- added J22, J24: 1S 1P -ve, TestPoint:TestPoint_Pad_D2.0mm, symbol Connector:Conn_01x01_Pin
Connections:
- net 1S_B- is gone; now on an unnamed net: J2.1 (Pin_1)
- net 1S_B+: no longer names the net of J1.1 (Pin_1)
- removed net 4P_B+: BT6.1 (+), BT7.1 (+), BT8.1 (+), BT9.1 (+), J10.1 (Pin_1), J12.1 (Pin_1), J14.1 (Pin_1), J16.1 (Pin_1)
- removed net 4P_B-: BT6.2 (-), BT7.2 (-), BT8.2 (-), BT9.2 (-), J11.1 (Pin_1), J13.1 (Pin_1), J15.1 (Pin_1), J17.1 (Pin_1)
- new net: J21.1 (Pin_1), J22.1 (Pin_1)
- new net: J23.1 (Pin_1), J24.1 (Pin_1)
- new net: BT7.2 (-), BT8.1 (+), J12.1 (Pin_1), J16.1 (Pin_1)
- new net: BT8.2 (-), BT9.1 (+), J13.1 (Pin_1), J15.1 (Pin_1)
- new net: BT6.2 (-), BT7.1 (+), J11.1 (Pin_1), J17.1 (Pin_1)
- new net: BT9.2 (-), J14.1 (Pin_1)
- new net: BT6.1 (+), J10.1 (Pin_1)
Other:
- note added: "PCB Track Resistance"
- note removed: "1S 1P MODULE (Single Cell ACIR Baseline)"
- note removed: "1S 4P MODULE (Parallel Current Sharing & R/4 ACIR Pack)"
- note removed: "Baseline 18650 EIS Measurement: ACIR = R_cell"
- moved on the sheet: BT7, BT9

Commit message: feat: add ACIR Learning Kit 2 PCB design files and production outputs
Parts:
- J10: value 1S 1P +ve -> 4S(II) B +ve
- J11: value 1S 1P -ve -> 4S(II) BT6 -ve
- J12: value 1S 3P +ve -> 4S(II) BT8 +ve
- J13: value 1S 3P -ve -> 4S(II) BT8 -ve
- J14: value 1S 4P +ve -> 4S(II) B -ve
- J15: value 1S 4P -ve -> 4S(II) BT9 +ve
- J16: value 1S 2P +ve -> 4S(II) BT7 -ve
- J17: value 1S 2P -ve -> 4S(II) BT7 +ve
- P1: renamed from J2; value 1S 1P -ve -> Track 1 Probe 1
- P2: renamed from J1; value 1S 1P +ve -> Track 1 Probe 2
- P3: renamed from J21; value 1S 1P +ve -> Track 2 Probe 1
- P4: renamed from J22; value 1S 1P -ve -> Track 2 Probe 2
- P5: renamed from J23; value 1S 1P +ve -> Track 3 Probe 1
- P6: renamed from J24; value 1S 1P -ve -> Track 3 Probe 2
Connections:
- net 4S2_MID2: now reaches BT7.2 (-), BT8.1 (+), J12.1 (Pin_1), J16.1 (Pin_1)
- net 4S2_MID3: now reaches BT8.2 (-), BT9.1 (+), J13.1 (Pin_1), J15.1 (Pin_1)
- net 4S2_MID1: now reaches BT6.2 (-), BT7.1 (+), J11.1 (Pin_1), J17.1 (Pin_1)
- net 4S2_B-: now reaches BT9.2 (-), J14.1 (Pin_1)
- net 4S2_B+: now reaches BT6.1 (+), J10.1 (Pin_1)
Other:
- note added: "4S 1P (II) MODULE (Varying Interconnect Track Resistance - Educational Pack Experiment)"
- note added: "Cells have IDENTICAL ACIR (~20mOhm). Series interconnects vary systematically: Link 1 (BT6-BT7): Ultra-wide 10mm 2-layer bus with dense via matrix (~0.5mOhm) Link 2 (BT7-BT8): Medium 3.0mm single-layer trace (~3.0mOhm) Link 3 (BT8-BT9): Narrow 0.8mm single-layer trace (~10.0mOhm) Demonstrates how interconnect trace impedance directly inflates total pack ACIR."
- note removed: "Individual cell branch test points (J10-J17) enable Kelvin characterization of each parallel cell & current sharing."
Changed lines of the file:
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@@
 		(company "Decibels Lab Pvt Ltd")
 		(comment 1 "Comprehensive 18650 ACIR Characterization Platform")
-		(comment 2 "Configurations: 1S 1P Baseline | 1S 4P Parallel Current Sharing | 4S 1P Series String")
+		(comment 2 "Kit 2: PCB Track Resistance | 4S1P (I) Differential ACIR | 4S1P (II) Varying Interconnect IR")
 		(comment 3 "High-Frequency 1kHz Kelvin 4-Wire EIS Sensing Architecture & Ultra-Dense Via Arrays")
 		(comment 4 "Production-Ready Hardware Design & Educational Measurement Kit")
@@
 		)
 	)
-	(text "Individual cell branch test points (J10-J17) enable Kelvin characterization of each parallel cell & current sharing."
-		(exclude_from_sim no)
-		(at 132.08 108 0)
-		(effects
-			(font
-				(size 1 1)
-			)
-			(justify left bottom)
-		)
-	)
 	(text "4-Wire Kelvin ACIR Measurement:"
 		(exclude_from_sim no)
@@
 	(wire
 		(pts
-			(xy 363.22 73.66) (xy 363.22 85.09)
-		)
-		(stroke
-			(width 0)
-			(type default)
-		)
-	)
-	(wire
-		(pts
 			(xy 101.6 180.34) (xy 101.6 193.04)
 		)
@@
 	(wire
 		(pts
-			(xy 261.62 58.42) (xy 261.62 66.04)
-		)
-		(stroke
-			(width 0)
-			(type default)
-		)
-	)
-	(wire
-		(pts
-			(xy 363.22 85.09) (xy 363.22 93.98)
-		)
-		(stroke
-			(width 0)
-			(type default)
-		)
-	)
-	(wire
-		(pts
 			(xy 101.6 166.37) (xy 132.08 166.37)
 		)
@@
 	(wire
 		(pts
-			(xy 312.42 58.42) (xy 312.42 66.04)
-		)
-		(stroke
-			(width 0)
-			(type default)
-		)
-	)
-	(wire
-		(pts
 			(xy 101.6 207.01) (xy 132.08 207.01)
 		)
@@
 	(wire
 		(pts
-			(xy 312.42 73.66) (xy 312.42 85.09)
-		)
-		(stroke
-			(width 0)
-			(type default)
-		)
-	)
-	(wire
-		(pts
 			(xy 101.6 147.32) (xy 101.6 152.4)
 		)
@@
 	(wire
 		(pts
-			(xy 261.62 73.66) (xy 261.62 83.82)
-		)
-		(stroke
-			(width 0)
-			(type default)
-		)
-	)
-	(wire
-		(pts
-			(xy 210.82 73.66) (xy 210.82 83.82)
-		)
-		(stroke
-			(width 0)
-			(type default)
-		)
-	)
-	(wire
-		(pts
-			(xy 363.22 48.26) (xy 363.22 66.04)
-		)
-		(stroke
-			(width 0)
-			(type default)
-		)
-	)
-	(wire
-		(pts
 			(xy 54.61 50.8) (xy 54.61 78.74)
 		)
@@
 	(wire
 		(pts
-			(xy 210.82 48.26) (xy 210.82 66.04)
-		)
-		(stroke
-			(width 0)
-			(type default)
-		)
-	)
-	(wire
-		(pts
-			(xy 261.62 48.26) (xy 261.62 58.42)
-		)
-		(stroke
-			(width 0)
-			(type default)
-		)
-	)
-	(wire
-		(pts
-			(xy 312.42 85.09) (xy 363.22 85.09)
-		)
-		(stroke
-			(width 0)
-			(type default)
-		)
-	)
-	(wire
-		(pts
 			(xy 73.66 50.8) (xy 73.66 78.74)
 		)
@@
 	(wire
 		(pts
-			(xy 261.62 58.42) (xy 312.42 58.42)
-		)
-		(stroke
-			(width 0)
-			(type default)
-		)
-	)
-	(wire
-		(pts
 			(xy 71.12 166.37) (xy 101.6 166.37)
 		)
@@
 	(wire
 		(pts
-			(xy 210.82 83.82) (xy 261.62 83.82)
-		)
-		(stroke
-			(width 0)
-			(type default)
-		)
-	)
-	(wire
-		(pts
 			(xy 93.98 50.8) (xy 93.98 78.74)
 		)
@@
 	(wire
 		(pts
-			(xy 312.42 48.26) (xy 312.42 58.42)
-		)
-		(stroke
-			(width 0)
-			(type default)
-		)
-	)
-	(wire
-		(pts
-			(xy 210.82 83.82) (xy 210.82 93.98)
-		)
-		(stroke
-			(width 0)
-			(type default)
-		)
-	)
-	(wire
-		(pts
 			(xy 71.12 186.69) (xy 101.6 186.69)
 		)
@@
 		)
 	)
-	(wire
-		(pts
-			(xy 312.42 85.09) (xy 312.42 93.98)
-		)
-		(stroke
-			(width 0)
-			(type default)
-		)
-	)
-	(wire
-		(pts
-			(xy 261.62 83.82) (xy 261.62 93.98)
-		)
-		(stroke
-			(width 0)
-			(type default)
-		)
-	)
 	(label "4S_B-"
 		(at 101.6 226.06 0)
@@
 		(dnp no)
 		(fields_autoplaced yes)
-		(property "Reference" "J22"
+		(property "Reference" "P4"
 			(at 97.79 82.55 270)
 			(show_name no)
@@
 			)
 		)
-		(property "Value" "1S 1P -ve"
+		(property "Value" "Track 2 Probe 2"
 			(at 97.79 85.09 270)
 			(show_name no)
@@
 		(dnp no)
 		(fields_autoplaced yes)
-		(property "Reference" "J23"
+		(property "Reference" "P5"
 			(at 58.42 44.45 90)
 			(show_name no)
@@
 			)
 		)
-		(property "Value" "1S 1P +ve"
+		(property "Value" "Track 3 Probe 1"
 			(at 58.42 46.99 90)
 			(show_name no)
@@
 			)
 		)
-		(property "Value" "1S 2P -ve"
+		(property "Value" "4S(II) BT7 +ve"
 			(at 265.43 100.33 270)
 			(show_name no)
@@
 			)
 		)
-		(property "Value" "1S 3P -ve"
+		(property "Value" "4S(II) BT8 -ve"
 			(at 316.23 100.33 270)
 			(show_name no)
@@
 		(dnp no)
 		(fields_autoplaced yes)
-		(property "Reference" "J2"
+		(property "Reference" "P1"
 			(at 77.47 82.55 270)
 			(show_name no)
@@
 			)
 		)
-		(property "Value" "1S 1P -ve"
+		(property "Value" "Track 1 Probe 1"
 			(at 77.47 85.09 270)
 			(show_name no)
@@
 			)
 		)
-		(property "Value" "1S 3P +ve"
+		(property "Value" "4S(II) BT8 +ve"
 			(at 316.23 44.45 90)
 			(show_name no)
@@
 		(dnp no)
 		(fields_autoplaced yes)
-		(property "Reference" "J24"
+		(property "Reference" "P6"
 			(at 58.42 82.55 270)
 			(show_name no)
@@
 			)
 		)
-		(property "Value" "1S 1P -ve"
+		(property "Value" "Track 3 Probe 2"
 			(at 58.42 85.09 270)
 			(show_name no)
@@
 			)
 		)
-		(property "Value" "1S 4P -ve"
+		(property "Value" "4S(II) BT9 +ve"
 			(at 367.03 100.33 270)
 			(show_name no)
@@
 			)
 		)
-		(property "Value" "1S 2P +ve"
+		(property "Value" "4S(II) BT7 -ve"
 			(at 265.43 44.45 90)
 			(show_name no)
@@
 			)
 		)
-		(property "Value" "1S 1P +ve"
+		(property "Value" "4S(II) B +ve"
 			(at 214.63 44.45 90)
 			(show_name no)
@@
 			)
 		)
-		(property "Value" "1S 4P +ve"
+		(property "Value" "4S(II) B -ve"
 			(at 367.03 44.45 90)
 			(show_name no)
@@
 			)
 		)
-		(property "Value" "1S 1P -ve"
+		(property "Value" "4S(II) BT6 -ve"
 			(at 214.63 100.33 270)
 			(show_name no)
@@
 		(dnp no)
 		(fields_autoplaced yes)
-		(property "Reference" "J21"
+		(property "Reference" "P3"
 			(at 97.79 44.45 90)
 			(show_name no)
@@
 			)
 		)
-		(property "Value" "1S 1P +ve"
+		(property "Value" "Track 2 Probe 1"
 			(at 97.79 46.99 90)
 			(show_name no)
@@
 		(dnp no)
 		(fields_autoplaced yes)
-		(property "Reference" "J1"
+		(property "Reference" "P2"
 			(at 77.47 44.45 90)
 			(show_name no)
@@
 			)
 		)
-		(property "Value" "1S 1P +ve"
+		(property "Value" "Track 1 Probe 2"
 			(at 77.47 46.99 90)
 			(show_name no)
@@
 	)
 	(embedded_fonts no)
+	(wire
+		(pts (xy 210.82 48.26) (xy 210.82 66.04))
+		(stroke (width 0) (type default))
+	)
+	(label "4S2_B+"
+		(at 210.82 58.42 0)
+		(effects (font (size 1.27 1.27)) (justify left))
+	)
+	(wire
+		(pts (xy 210.82 73.66) (xy 210.82 93.98))
+		(stroke (width 0) (type default))
+	)
+	(wire
+		(pts (xy 210.82 83.82) (xy 261.62 83.82))
+		(stroke (width 0) (type default))
+	)
+	(wire
+		(pts (xy 261.62 73.66) (xy 261.62 93.98))
+		(stroke (width 0) (type default))
+	)
+	(label "4S2_MID1"
+		(at 236.22 83.82 0)
+		(effects (font (size 1.27 1.27)) (justify left))
+	)
+	(wire
+		(pts (xy 261.62 48.26) (xy 261.62 66.04))
+		(stroke (width 0) (type default))
+	)
+	(wire
+		(pts (xy 261.62 58.42) (xy 312.42 58.42))
+		(stroke (width 0) (type default))
+	)
+	(wire
+		(pts (xy 312.42 48.26) (xy 312.42 66.04))
+		(stroke (width 0) (type default))
+	)
+	(label "4S2_MID2"
+		(at 287.02 58.42 0)
+		(effects (font (size 1.27 1.27)) (justify left))
+	)
+	(wire
+		(pts (xy 312.42 73.66) (xy 312.42 93.98))
+		(stroke (width 0) (type default))
+	)
+	(wire
+		(pts (xy 312.42 85.09) (xy 363.22 85.09))
+		(stroke (width 0) (type default))
+	)
+	(wire
+		(pts (xy 363.22 73.66) (xy 363.22 93.98))
+		(stroke (width 0) (type default))
+	)
+	(label "4S2_MID3"
+		(at 337.82 85.09 0)
+		(effects (font (size 1.27 1.27)) (justify left))
+	)
+	(wire
+		(pts (xy 363.22 48.26) (xy 363.22 66.04))
+		(stroke (width 0) (type default))
+	)
+	(label "4S2_B-"
+		(at 363.22 58.42 0)
+		(effects (font (size 1.27 1.27)) (justify left))
+	)
+	(text "4S 1P (II) MODULE (Varying Interconnect Track Resistance - Educational Pack Experiment)"
+		(at 200 35 0)
+		(effects (font (size 2 2) (bold yes)) (justify left))
+	)
+	(text "Cells have IDENTICAL ACIR (~20mOhm). Series interconnects vary systematically:\nLink 1 (BT6-BT7): Ultra-wide 10mm 2-layer bus with dense via matrix (~0.5mOhm)\nLink 2 (BT7-BT8): Medium 3.0mm single-layer trace (~3.0mOhm)\nLink 3 (BT8-BT9): Narrow 0.8mm single-layer trace (~10.0mOhm)\nDemonstrates how interconnect trace impedance directly inflates total pack ACIR."
+		(at 200 115 0)
+		(effects (font (size 1.27 1.27)) (justify left))
+	)
 )

Commit message: feat: DFM optimization - clean circular probing pads, uniform 2.0mm via pitch, and zero warnings
Parts:
- J10, J11, J12, J13, J14, J15, J16, J17, J18, J19, J20, J3, J4, J7, J8, J9, P1, P2, P3, P4, P5, P6: footprint TestPoint:TestPoint_Pad_D2.0mm -> footprints:TestPoint_Pad_D6.0mm
Changed lines of the file:
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@@
 			)
 		)
-		(property "Footprint" "TestPoint:TestPoint_Pad_D2.0mm"
+		(property "Footprint" "footprints:TestPoint_Pad_D6.0mm"
 			(at 137.16 207.01 0)
 			(hide yes)
@@
 			)
 		)
-		(property "Footprint" "TestPoint:TestPoint_Pad_D2.0mm"
+		(property "Footprint" "footprints:TestPoint_Pad_D6.0mm"
 			(at 93.98 83.82 0)
 			(hide yes)
@@
 			)
 		)
-		(property "Footprint" "TestPoint:TestPoint_Pad_D2.0mm"
+		(property "Footprint" "footprints:TestPoint_Pad_D6.0mm"
 			(at 54.61 45.72 0)
 			(hide yes)
@@
 			)
 		)
-		(property "Footprint" "TestPoint:TestPoint_Pad_D2.0mm"
+		(property "Footprint" "footprints:TestPoint_Pad_D6.0mm"
 			(at 261.62 99.06 0)
 			(hide yes)
@@
 			)
 		)
-		(property "Footprint" "TestPoint:TestPoint_Pad_D2.0mm"
+		(property "Footprint" "footprints:TestPoint_Pad_D6.0mm"
 			(at 101.6 142.24 0)
 			(hide yes)
@@
 			)
 		)
-		(property "Footprint" "TestPoint:TestPoint_Pad_D2.0mm"
+		(property "Footprint" "footprints:TestPoint_Pad_D6.0mm"
 			(at 66.04 186.69 0)
 			(hide yes)
@@
 			)
 		)
-		(property "Footprint" "TestPoint:TestPoint_Pad_D2.0mm"
+		(property "Footprint" "footprints:TestPoint_Pad_D6.0mm"
 			(at 101.6 233.68 0)
 			(hide yes)
@@
 			)
 		)
-		(property "Footprint" "TestPoint:TestPoint_Pad_D2.0mm"
+		(property "Footprint" "footprints:TestPoint_Pad_D6.0mm"
 			(at 66.04 207.01 0)
 			(hide yes)
@@
 			)
 		)
-		(property "Footprint" "TestPoint:TestPoint_Pad_D2.0mm"
+		(property "Footprint" "footprints:TestPoint_Pad_D6.0mm"
 			(at 312.42 99.06 0)
 			(hide yes)
@@
 			)
 		)
-		(property "Footprint" "TestPoint:TestPoint_Pad_D2.0mm"
+		(property "Footprint" "footprints:TestPoint_Pad_D6.0mm"
 			(at 137.16 166.37 0)
 			(hide yes)
@@
 			)
 		)
-		(property "Footprint" "TestPoint:TestPoint_Pad_D2.0mm"
+		(property "Footprint" "footprints:TestPoint_Pad_D6.0mm"
 			(at 73.66 83.82 0)
 			(hide yes)
@@
 			)
 		)
-		(property "Footprint" "TestPoint:TestPoint_Pad_D2.0mm"
+		(property "Footprint" "footprints:TestPoint_Pad_D6.0mm"
 			(at 312.42 43.18 0)
 			(hide yes)
@@
 			)
 		)
-		(property "Footprint" "TestPoint:TestPoint_Pad_D2.0mm"
+		(property "Footprint" "footprints:TestPoint_Pad_D6.0mm"
 			(at 54.61 83.82 0)
 			(hide yes)
@@
 			)
 		)
-		(property "Footprint" "TestPoint:TestPoint_Pad_D2.0mm"
+		(property "Footprint" "footprints:TestPoint_Pad_D6.0mm"
 			(at 363.22 99.06 0)
 			(hide yes)
@@
 			)
 		)
-		(property "Footprint" "TestPoint:TestPoint_Pad_D2.0mm"
+		(property "Footprint" "footprints:TestPoint_Pad_D6.0mm"
 			(at 261.62 43.18 0)
 			(hide yes)
@@
 			)
 		)
-		(property "Footprint" "TestPoint:TestPoint_Pad_D2.0mm"
+		(property "Footprint" "footprints:TestPoint_Pad_D6.0mm"
 			(at 210.82 43.18 0)
 			(hide yes)
@@
 			)
 		)
-		(property "Footprint" "TestPoint:TestPoint_Pad_D2.0mm"
+		(property "Footprint" "footprints:TestPoint_Pad_D6.0mm"
 			(at 137.16 186.69 0)
 			(hide yes)
@@
 			)
 		)
-		(property "Footprint" "TestPoint:TestPoint_Pad_D2.0mm"
+		(property "Footprint" "footprints:TestPoint_Pad_D6.0mm"
 			(at 363.22 43.18 0)
 			(hide yes)
@@
 			)
 		)
-		(property "Footprint" "TestPoint:TestPoint_Pad_D2.0mm"
+		(property "Footprint" "footprints:TestPoint_Pad_D6.0mm"
 			(at 210.82 99.06 0)
 			(hide yes)
@@
 			)
 		)
-		(property "Footprint" "TestPoint:TestPoint_Pad_D2.0mm"
+		(property "Footprint" "footprints:TestPoint_Pad_D6.0mm"
 			(at 66.04 166.37 0)
 			(hide yes)
@@
 			)
 		)
-		(property "Footprint" "TestPoint:TestPoint_Pad_D2.0mm"
+		(property "Footprint" "footprints:TestPoint_Pad_D6.0mm"
 			(at 93.98 45.72 0)
 			(hide yes)
@@
 			)
 		)
-		(property "Footprint" "TestPoint:TestPoint_Pad_D2.0mm"
+		(property "Footprint" "footprints:TestPoint_Pad_D6.0mm"
 			(at 73.66 45.72 0)
 			(hide yes)
