File: ACIR-Learning-Kit-2-PCB/ACIR-Learning-Kit-2-PCB.kicad_pcb (KiCad board)
At the start: 2 copper layers, 297 x 210 mm, 40 parts, among them J10 1S 1P +ve, J11 1S 1P -ve, J12 1S 3P +ve, J13 1S 3P -ve, J14 1S 4P +ve, J15 1S 4P -ve, J16 1S 2P +ve, J17 1S 2P -ve, J18 1S 1P -ve, J19 2S 1P -ve, J20 3S 1P -ve, J3 4S B +ve, J4 4S B -ve, J7 2S 1P +ve, J8 3S 1P +ve, J9 4S 1P +ve, P1 1S 1P -ve, P2 1S 1P +ve, P3 1S 1P +ve, P4 1S 1P -ve, P5 1S 1P +ve, P6 1S 1P -ve

Commit message: feat: add PCB design files, gerbers, and production outputs for ACIR Learning Kits 1 and 2
Routing:
- net Net-(BT8--): track 177.5 -> 152.9 mm
- net Net-(BT7--): track 263.0 -> 238.4 mm
Changed lines of the file:
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@@
 			(pintype "passive")
 		)
-		(pad "1" thru_hole circle
-			(at 36.11 0)
-			(size 3.5 3.5)
-			(drill 2.5)
-			(layers "*.Cu" "*.Mask")
-			(remove_unused_layers no)
-			(net "Net-(BT7--)")
-			(pinfunction "+_1")
-			(pintype "passive")
-		)
 		(pad "1" smd rect
 			(at 39.63 0 90)
@@
 			(pintype "passive")
 		)
-		(pad "2" thru_hole circle
-			(at -36.11 0)
-			(size 3.5 3.5)
-			(drill 2.5)
-			(layers "*.Cu" "*.Mask")
-			(remove_unused_layers no)
-			(net "Net-(BT8--)")
-			(pinfunction "-_2")
-			(pintype "passive")
-		)
 		(pad "2" thru_hole oval
 			(at -28.35 0)
@@
 			(pintype "passive")
 		)
-		(pad "1" thru_hole circle
-			(at 36.11 0)
-			(size 3.5 3.5)
-			(drill 2.5)
-			(layers "*.Cu" "*.Mask")
-			(remove_unused_layers no)
-			(net "Net-(BT3--)")
-			(pinfunction "+_1")
-			(pintype "passive")
-		)
 		(pad "1" smd rect
 			(at 39.63 0 90)
@@
 			(pintype "passive")
 		)
-		(pad "2" thru_hole circle
-			(at -36.11 0)
-			(size 3.5 3.5)
-			(drill 2.5)
-			(layers "*.Cu" "*.Mask")
-			(remove_unused_layers no)
-			(net "Net-(BT4--)")
-			(pinfunction "-_2")
-			(pintype "passive")
-		)
 		(pad "2" thru_hole oval
 			(at -28.35 0)
@@
 			(pintype "passive")
 		)
-		(pad "1" thru_hole circle
-			(at 36.11 0 180)
-			(size 3.5 3.5)
-			(drill 2.5)
-			(layers "*.Cu" "*.Mask")
-			(remove_unused_layers no)
-			(net "Net-(BT6--)")
-			(pinfunction "+_1")
-			(pintype "passive")
-		)
 		(pad "1" smd rect
 			(at 39.63 0 270)
@@
 			(pintype "passive")
 		)
-		(pad "2" thru_hole circle
-			(at -36.11 0 180)
-			(size 3.5 3.5)
-			(drill 2.5)
-			(layers "*.Cu" "*.Mask")
-			(remove_unused_layers no)
-			(net "Net-(BT7--)")
-			(pinfunction "-_2")
-			(pintype "passive")
-		)
 		(pad "2" thru_hole oval
 			(at -28.35 0 180)
@@
 			(pintype "passive")
 		)
-		(pad "1" thru_hole circle
-			(at 36.11 0 180)
-			(size 3.5 3.5)
-			(drill 2.5)
-			(layers "*.Cu" "*.Mask")
-			(remove_unused_layers no)
-			(net "Net-(BT8--)")
-			(pinfunction "+_1")
-			(pintype "passive")
-		)
 		(pad "1" smd rect
 			(at 39.63 0 270)
@@
 			(pintype "passive")
 		)
-		(pad "2" thru_hole circle
-			(at -36.11 0 180)
-			(size 3.5 3.5)
-			(drill 2.5)
-			(layers "*.Cu" "*.Mask")
-			(remove_unused_layers no)
-			(net "Net-(BT9--)")
-			(pinfunction "-_2")
-			(pintype "passive")
-		)
 		(pad "2" thru_hole oval
 			(at -28.35 0 180)
@@
 			(pintype "passive")
 		)
-		(pad "1" thru_hole circle
-			(at 36.11 0)
-			(size 3.5 3.5)
-			(drill 2.5)
-			(layers "*.Cu" "*.Mask")
-			(remove_unused_layers no)
-			(net "/4S_B+")
-			(pinfunction "+_1")
-			(pintype "passive")
-		)
 		(pad "1" smd rect
 			(at 39.63 0 90)
@@
 			(pintype "passive")
 		)
-		(pad "2" thru_hole circle
-			(at -36.11 0)
-			(size 3.5 3.5)
-			(drill 2.5)
-			(layers "*.Cu" "*.Mask")
-			(remove_unused_layers no)
-			(net "Net-(BT2--)")
-			(pinfunction "-_2")
-			(pintype "passive")
-		)
 		(pad "2" thru_hole oval
 			(at -28.35 0)
@@
 			(pintype "passive")
 		)
-		(pad "1" thru_hole circle
-			(at 36.11 0 180)
-			(size 3.5 3.5)
-			(drill 2.5)
-			(layers "*.Cu" "*.Mask")
-			(remove_unused_layers no)
-			(net "Net-(BT4--)")
-			(pinfunction "+_1")
-			(pintype "passive")
-		)
 		(pad "1" smd rect
 			(at 39.63 0 270)
@@
 			(pintype "passive")
 		)
-		(pad "2" thru_hole circle
-			(at -36.11 0 180)
-			(size 3.5 3.5)
-			(drill 2.5)
-			(layers "*.Cu" "*.Mask")
-			(remove_unused_layers no)
-			(net "/4S_B-")
-			(pinfunction "-_2")
-			(pintype "passive")
-		)
 		(pad "2" thru_hole oval
 			(at -28.35 0 180)
@@
 			(pintype "passive")
 		)
-		(pad "1" thru_hole circle
-			(at 36.11 0 180)
-			(size 3.5 3.5)
-			(drill 2.5)
-			(layers "*.Cu" "*.Mask")
-			(remove_unused_layers no)
-			(net "Net-(BT2--)")
-			(pinfunction "+_1")
-			(pintype "passive")
-		)
 		(pad "1" smd rect
 			(at 39.63 0 270)
@@
 			(pintype "passive")
 		)
-		(pad "2" thru_hole circle
-			(at -36.11 0 180)
-			(size 3.5 3.5)
-			(drill 2.5)
-			(layers "*.Cu" "*.Mask")
-			(remove_unused_layers no)
-			(net "Net-(BT3--)")
-			(pinfunction "-_2")
-			(pintype "passive")
-		)
 		(pad "2" thru_hole oval
 			(at -28.35 0 180)
@@
 			(pintype "passive")
 		)
-		(pad "1" thru_hole circle
-			(at 36.11 0)
-			(size 3.5 3.5)
-			(drill 2.5)
-			(layers "*.Cu" "*.Mask")
-			(remove_unused_layers no)
-			(net "Net-(BT6-+)")
-			(pinfunction "+_1")
-			(pintype "passive")
-		)
 		(pad "1" smd rect
 			(at 39.63 0 90)
@@
 			(pintype "passive")
 		)
-		(pad "2" thru_hole circle
-			(at -36.11 0)
-			(size 3.5 3.5)
-			(drill 2.5)
-			(layers "*.Cu" "*.Mask")
-			(remove_unused_layers no)
-			(net "Net-(BT6--)")
-			(pinfunction "-_2")
-			(pintype "passive")
-		)
 		(pad "2" thru_hole oval
 			(at -28.35 0)
@@
 	)
 	(segment
-		(start 102.74 210.53)
-		(end 90.45 210.53)
-		(width 8)
-		(layer "B.Cu")
-		(net "Net-(BT8--)")
-	)
-	(segment
 		(start 105.28 189.32)
 		(end 102.74 186.78)
@@
 	)
 	(segment
-		(start 102.74 186.78)
-		(end 90.45 186.78)
-		(width 8)
-		(layer "B.Cu")
-		(net "Net-(BT8--)")
-	)
-	(segment
 		(start 105.28 184.24)
 		(end 105.28 189.32)
@@
 	)
 	(segment
-		(start 150.38 163.03)
-		(end 162.67 163.03)
-		(width 8)
-		(layer "B.Cu")
-		(net "Net-(BT7--)")
-	)
-	(segment
 		(start 147.84 189.32)
 		(end 147.84 184.24)
@@
 		(width 8)
 		(layer "B.Cu")
-		(net "Net-(BT7--)")
-	)
-	(segment
-		(start 150.38 186.78)
-		(end 162.67 186.78)
-		(width 8)
-		(layer "B.Cu")
